Commit message: Update nybble.urdf
Corrected weights and inertia. (Closer to real values)

File: nybble.urdf (robot description, URDF)
Before this commit: robot Nybble, 9 links, 8 joints
Links:
- link left_lower_arm: mass 0.1 -> 0.075
- link left_lower_leg: mass 0.1 -> 0.075
- link left_upper_arm: mass 0.1 -> 0.025
- link left_upper_leg: mass 0.1 -> 0.025
- link right_lower_arm: mass 0.1 -> 0.075
- link right_lower_leg: mass 0.1 -> 0.075
- link right_upper_arm: mass 0.1 -> 0.025
- link right_upper_leg: mass 0.1 -> 0.025
- link torso: mass 0.5 -> 0.2
Joints:
- joint elbow_left: limit lower=-3 upper=3 effort=2.0 velocity=5 -> lower=-1.57 upper=1.57 effort=0 velocity=0
- joint elbow_right: limit lower=-3 upper=3 effort=2.0 velocity=5 -> lower=-1.57 upper=1.57 effort=0 velocity=0
- joint hip_left: limit lower=-3 upper=3 effort=2.0 velocity=5 -> lower=-1.57 upper=1.57 effort=0 velocity=0
- joint hip_right: limit lower=-3 upper=3 effort=2.0 velocity=5 -> lower=-1.57 upper=1.57 effort=0 velocity=0
- joint knee_left: limit lower=-3 upper=3 effort=2.0 velocity=5 -> lower=-1.57 upper=1.57 effort=0 velocity=0
- joint knee_right: limit lower=-3 upper=3 effort=2.0 velocity=5 -> lower=-1.57 upper=1.57 effort=0 velocity=0
- joint shoulder_left: limit lower=-3 upper=3 effort=2.0 velocity=5 -> lower=-1.57 upper=1.57 effort=0 velocity=0
- joint shoulder_right: limit lower=-3 upper=3 effort=2.0 velocity=5 -> lower=-1.57 upper=1.57 effort=0 velocity=0
